Commit message: add support for gazebo classic

File: robotiq_description/urdf/2f_140.ros2_control.xacro (robot description, xacro)
@@ -4,4 +4,5 @@
         name
         prefix
+        sim_gazebo:=false
         sim_ignition:=false
         sim_isaac:=false
@@ -14,4 +15,7 @@
             <!-- Plugins -->
             <hardware>
+                <xacro:if value="${sim_gazebo}">
+                    <plugin>gazebo_ros2_control/GazeboSystem</plugin>
+                </xacro:if>
                 <xacro:if value="${sim_isaac}">
                     <plugin>topic_based_ros2_control/TopicBasedSystem</plugin>
@@ -45,5 +49,5 @@
             </joint>
             <!-- When simulating we need to include the rest of the gripper joints -->
-            <xacro:if value="${use_fake_hardware or sim_isaac or sim_ignition}">
+            <xacro:if value="${use_fake_hardware or sim_isaac or sim_ignition or sim_gazebo}">
                 <joint name="${prefix}left_inner_knuckle_joint">
                     <param name="mimic">${prefix}finger_joint</param>
@@ -93,5 +97,5 @@
             </xacro:if>
             <!-- Only add this with fake hardware mode -->
-            <xacro:unless value="${sim_ignition or sim_isaac}">
+            <xacro:unless value="${sim_gazebo or sim_ignition or sim_isaac}">
                 <gpio name="reactivate_gripper">
                     <command_interface name="reactivate_gripper_cmd" />

File: robotiq_description/urdf/2f_85.ros2_control.xacro (robot description, xacro)
@@ -4,4 +4,5 @@
         name
         prefix
+        sim_gazebo:=false
         sim_ignition:=false
         sim_isaac:=false
@@ -16,4 +17,7 @@
                 <!-- Set use_dummy to true to connect to a dummy driver for testing purposes. -->
                 <param name="use_dummy">false</param>
+                <xacro:if value="${sim_gazebo}">
+                    <plugin>gazebo_ros2_control/GazeboSystem</plugin>
+                </xacro:if>
                 <xacro:if value="${sim_isaac}">
                     <plugin>topic_based_ros2_control/TopicBasedSystem</plugin>
@@ -48,5 +52,5 @@
             </joint>
             <!-- When simulating we need to include the rest of the gripper joints -->
-            <xacro:if value="${use_fake_hardware or sim_isaac or sim_ignition}">
+            <xacro:if value="${use_fake_hardware or sim_isaac or sim_ignition or sim_gazebo}">
                 <joint name="${prefix}robotiq_85_right_knuckle_joint">
                     <param name="mimic">${prefix}robotiq_85_left_knuckle_joint</param>
@@ -96,5 +100,5 @@
             </xacro:if>
             <!-- Only add this with fake hardware mode -->
-            <xacro:unless value="${sim_ignition or sim_isaac}">
+            <xacro:unless value="${sim_gazebo or sim_ignition or sim_isaac}">
                 <gpio name="reactivate_gripper">
                     <command_interface name="reactivate_gripper_cmd" />

File: robotiq_description/urdf/robotiq_2f_140_macro.urdf.xacro (robot description, xacro)
@@ -6,4 +6,5 @@
         parent
         *origin
+        sim_gazebo:=false
         sim_ignition:=false
         sim_isaac:=false
@@ -20,4 +21,5 @@
             <xacro:robotiq_gripper_ros2_control
                 name="${name}" prefix="${prefix}"
+                sim_gazebo="${sim_gazebo}"
                 sim_ignition="${sim_ignition}"
                 sim_isaac="${sim_isaac}"
@@ -68,4 +70,31 @@
       <xacro:finger_joint prefix="${prefix}"/>
       <xacro:right_outer_knuckle_joint prefix="${prefix}"/>
+      <!-- fix "_mimic" joint interface name suffix causes Moveit2 "Joint not found" Error -->
+      <!-- https://github.com/ros-controls/gazebo_ros2_control/issues/173 -->
+      <link name="${prefix}dummy_child1"/>
+      <link name="${prefix}dummy_child2"/>
+      <link name="${prefix}dummy_child3"/>
+      <link name="${prefix}dummy_child4"/>
+      <link name="${prefix}dummy_child5"/>
+      <joint name="${prefix}left_inner_knuckle_joint_mimic" type="fixed">
+        <parent link="${prefix}robotiq_140_base_link" />
+        <child link="${prefix}dummy_child1" />
+      </joint>
+      <joint name="${prefix}left_inner_finger_joint_mimic" type="fixed">
+        <parent link="${prefix}robotiq_140_base_link" />
+        <child link="${prefix}dummy_child2" />
+      </joint>
+      <joint name="${prefix}right_outer_knuckle_joint_mimic" type="fixed">
+        <parent link="${prefix}robotiq_140_base_link" />
+        <child link="${prefix}dummy_child3" />
+      </joint>
+      <joint name="${prefix}right_inner_knuckle_joint_mimic" type="fixed">
+        <parent link="${prefix}robotiq_140_base_link" />
+        <child link="${prefix}dummy_child4" />
+      </joint>
+      <joint name="${prefix}right_inner_finger_joint_mimic" type="fixed">
+        <parent link="${prefix}robotiq_140_base_link" />
+        <child link="${prefix}dummy_child5" />
+      </joint>
     </xacro:macro>
 </robot>

File: robotiq_description/urdf/robotiq_2f_85_macro.urdf.xacro (robot description, xacro)
@@ -6,4 +6,5 @@
         parent
         *origin
+        sim_gazebo:=false
         sim_ignition:=false
         sim_isaac:=false
@@ -20,4 +21,5 @@
             <xacro:robotiq_gripper_ros2_control
                 name="${name}" prefix="${prefix}"
+                sim_gazebo="${sim_gazebo}"
                 sim_ignition="${sim_ignition}"
                 sim_isaac="${sim_isaac}"
@@ -275,4 +277,31 @@
             <mimic joint="${prefix}robotiq_85_left_knuckle_joint" />
         </joint>
+        <!-- fix "_mimic" joint interface name suffix causes Moveit2 "Joint not found" Error -->
+        <!-- https://github.com/ros-controls/gazebo_ros2_control/issues/173 -->
+        <link name="${prefix}dummy_child1"/>
+        <link name="${prefix}dummy_child2"/>
+        <link name="${prefix}dummy_child3"/>
+        <link name="${prefix}dummy_child4"/>
+        <link name="${prefix}dummy_child5"/>
+        <joint name="${prefix}robotiq_85_right_knuckle_joint_mimic" type="fixed">
+            <parent link="${prefix}robotiq_85_base_link" />
+            <child link="${prefix}dummy_child1" />
+        </joint>
+        <joint name="${prefix}robotiq_85_left_inner_knuckle_joint_mimic" type="fixed">
+            <parent link="${prefix}robotiq_85_base_link" />
+            <child link="${prefix}dummy_child2" />
+        </joint>
+        <joint name="${prefix}robotiq_85_right_inner_knuckle_joint_mimic" type="fixed">
+            <parent link="${prefix}robotiq_85_base_link" />
+            <child link="${prefix}dummy_child3" />
+        </joint>
+        <joint name="${prefix}robotiq_85_left_finger_tip_joint_mimic" type="fixed">
+            <parent link="${prefix}robotiq_85_base_link" />
+            <child link="${prefix}dummy_child4" />
+        </joint>
+        <joint name="${prefix}robotiq_85_right_finger_tip_joint_mimic" type="fixed">
+            <parent link="${prefix}robotiq_85_base_link" />
+            <child link="${prefix}dummy_child5" />
+        </joint>
     </xacro:macro>
 </robot>
