Commit message: add grasp fix

File: robotiq_description/urdf/robotiq_2f_85_gripper.gazebo.urdf.xacro (robot description, xacro)
@@ -13,5 +13,5 @@
         parent="world"
         sim_gazebo="true">
-        <origin xyz="0 0 0" rpy="0 0 0" />
+        <origin xyz="0 0 0.3" rpy="0 0 0" />
     </xacro:robotiq_gripper>
     <gazebo>

File: robotiq_description/urdf/robotiq_2f_85_macro.urdf.xacro (robot description, xacro)
@@ -14,5 +14,6 @@
         fake_sensor_commands:=false
         include_ros2_control:=true
-        com_port:=/dev/ttyUSB0">
+        com_port:=/dev/ttyUSB0
+        palm_link:=robotiq_85_base_link">
         <!-- ros2 control include -->
         <xacro:include filename="$(find robotiq_description)/urdf/2f_85.ros2_control.xacro" />
@@ -304,4 +305,28 @@
             <child link="${prefix}dummy_child5" />
         </joint>
+        <!-- grasp fix plugin for gazebo classic -->
+        <xacro:if value="${sim_gazebo}">
+            <gazebo>
+                <plugin name="gazebo_grasp_fix" filename="libgazebo_grasp_fix.so">
+                    <arm>
+                        <arm_name>${prefix}robotiq_85_gripper_arm</arm_name>
+                        <palm_link>${prefix}${palm_link}</palm_link>
+                        <gripper_link>${prefix}robotiq_85_left_finger_tip_link</gripper_link>
+                        <gripper_link>${prefix}robotiq_85_right_finger_tip_link</gripper_link>
+                        <gripper_link>${prefix}robotiq_85_left_knuckle_link</gripper_link>
+                        <gripper_link>${prefix}robotiq_85_right_knuckle_link</gripper_link>
+                        <gripper_link>${prefix}robotiq_85_left_inner_knuckle_link</gripper_link>
+                        <gripper_link>${prefix}robotiq_85_right_inner_knuckle_link</gripper_link>
+                    </arm>
+                    <forces_angle_tolerance>150</forces_angle_tolerance>
+                    <update_rate>30</update_rate>
+                    <grip_count_threshold>1</grip_count_threshold>
+                    <max_grip_count>2</max_grip_count>
+                    <release_tolerance>0.01</release_tolerance>
+                    <disable_collisions_on_attach>false</disable_collisions_on_attach>
+                    <contact_topic>__default_topic__</contact_topic>
+                 </plugin>
+             </gazebo>
+        </xacro:if>
     </xacro:macro>
 </robot>
