Commit message: move gazebo ros control plugin outside the macro, change 3d files loading

File: robotiq_description/urdf/robotiq_2f_85_gripper.urdf.xacro (robot description, xacro)
@@ -15,3 +15,13 @@
         <origin xyz="0 0 0.3" rpy="0 0 0" />
     </xacro:robotiq_2f_85_gripper>
+    <xacro:if value="$(arg sim_gazebo)">
+        <gazebo reference="world">
+        </gazebo>
+        <gazebo>
+            <!-- gazebo ros2 control plugin -->
+            <plugin name="gazebo_ros_control" filename="libgazebo_ros2_control.so">
+                <parameters>$(find robotiq_description)/config/robotiq_2f_85_controllers.yaml</parameters>
+            </plugin>
+        </gazebo>
+    </xacro:if>
 </robot>

File: robotiq_description/urdf/robotiq_2f_85_macro.urdf.xacro (robot description, xacro)
@@ -327,8 +327,4 @@
                     <contact_topic>__default_topic__</contact_topic>
                  </plugin>
-                 <!-- gazebo ros2 control plugin -->
-                 <plugin name="robotiq_2f_85_gazebo_ros_control" filename="libgazebo_ros2_control.so">
-                    <parameters>$(find robotiq_description)/config/robotiq_2f_85_controllers.yaml</parameters>
-                </plugin>
              </gazebo>
         </xacro:if>

File: robotiq_description/urdf/test_2f_85.urdf (robot description, URDF)
Before this commit: robot robotiq_gripper, 15 links, 14 joints
Joints:
- joint robotiq_85_base_joint: origin xyz=0 0 0 rpy=0 0 0 -> xyz=0 0 0.3 rpy=0 0 0
