Commit message: grasp in gazebo

File: robotiq_description/srdf/robotiq_2f_85_macro.srdf.xacro (robot description, xacro)
@@ -2,5 +2,5 @@
 <robot xmlns:xacro="http://wiki.ros.org/xacro">
     <xacro:macro name="robotiq_2f_85_srdf" params="prefix">
-        <group name="${prefix}gripper">
+        <group name="${prefix}robotiq_2f_85_gripper">
             <link name="${prefix}robotiq_85_base_link"/>
             <link name="${prefix}robotiq_85_left_inner_knuckle_link"/>
@@ -12,10 +12,16 @@
             <link name="${prefix}robotiq_85_right_finger_link"/>
             <link name="${prefix}robotiq_85_right_finger_tip_link"/>
+            <joint name="${prefix}robotiq_85_left_knuckle_joint" />
+            <passive_joint name="${prefix}robotiq_85_right_knuckle_joint" />
+            <passive_joint name="${prefix}robotiq_85_left_inner_knuckle_joint" />
+            <passive_joint name="${prefix}robotiq_85_right_inner_knuckle_joint" />
+            <passive_joint name="${prefix}robotiq_85_left_finger_tip_joint" />
+            <passive_joint name="${prefix}robotiq_85_right_finger_tip_joint" />
         </group>
         <!--GROUP STATES - Purpose - Define a named state for a particular group, in terms of joint values. This is useful to define states like 'folded arms'-->
-        <group_state name="${prefix}open" group="${prefix}gripper">
+        <group_state name="${prefix}open" group="${prefix}robotiq_2f_85_gripper">
             <joint name="${prefix}robotiq_85_left_knuckle_joint" value="0" />
         </group_state>
-        <group_state name="${prefix}close" group="${prefix}gripper">
+        <group_state name="${prefix}close" group="${prefix}robotiq_2f_85_gripper">
             <joint name="${prefix}robotiq_85_left_knuckle_joint" value="0.7" />
         </group_state>

File: robotiq_description/urdf/robotiq_2f_140_macro.urdf.xacro (robot description, xacro)
@@ -1,5 +1,5 @@
 <?xml version="1.0"?>
 <robot xmlns:xacro="http://wiki.ros.org/xacro" name="robotiq_gripper">
-  <xacro:macro name="robotiq_gripper" params="
+  <xacro:macro name="robotiq_2f_140_gripper" params="
         name
         prefix

File: robotiq_description/urdf/robotiq_2f_85_gripper.urdf.xacro (robot description, xacro)
@@ -1,11 +1,17 @@
 <?xml version="1.0"?>
-<robot xmlns:xacro="http://wiki.ros.org/xacro" name="robotiq_gripper">
+<robot xmlns:xacro="http://wiki.ros.org/xacro" name="robotiq_2f_85_gripper">
     <!-- parameters -->
     <xacro:arg name="use_fake_hardware" default="true" />
+    <xacro:arg name="sim_gazebo" default="false"/>
+    <xacro:arg name="prefix" default="" />
     <!-- Import macros -->
     <xacro:include filename="$(find robotiq_description)/urdf/robotiq_2f_85_macro.urdf.xacro" />
     <link name="world" />
-    <xacro:robotiq_gripper name="RobotiqGripperHardwareInterface" prefix="" parent="world" use_fake_hardware="$(arg use_fake_hardware)">
-        <origin xyz="0 0 0" rpy="0 0 0" />
-    </xacro:robotiq_gripper>
+    <xacro:robotiq_2f_85_gripper name="RobotiqGripperHardwareInterface"
+        prefix="$(arg prefix)"
+        parent="world"
+        use_fake_hardware="$(arg use_fake_hardware)"
+        sim_gazebo="$(arg sim_gazebo)">
+        <origin xyz="0 0 0.3" rpy="0 0 0" />
+    </xacro:robotiq_2f_85_gripper>
 </robot>

File: robotiq_description/urdf/robotiq_2f_85_macro.urdf.xacro (robot description, xacro)
@@ -1,5 +1,5 @@
 <?xml version="1.0"?>
 <robot xmlns:xacro="http://wiki.ros.org/xacro" name="robotiq_gripper">
-    <xacro:macro name="robotiq_gripper" params="
+    <xacro:macro name="robotiq_2f_85_gripper" params="
         name
         prefix
@@ -305,7 +305,7 @@
             <child link="${prefix}dummy_child5" />
         </joint>
-        <!-- grasp fix plugin for gazebo classic -->
         <xacro:if value="${sim_gazebo}">
             <gazebo>
+                <!-- grasp fix plugin for gazebo classic -->
                 <plugin name="gazebo_grasp_fix" filename="libgazebo_grasp_fix.so">
                     <arm>
@@ -327,4 +327,8 @@
                     <contact_topic>__default_topic__</contact_topic>
                  </plugin>
+                 <!-- gazebo ros2 control plugin -->
+                 <plugin name="robotiq_2f_85_gazebo_ros_control" filename="libgazebo_ros2_control.so">
+                    <parameters>$(find robotiq_description)/config/robotiq_2f_85_controllers.yaml</parameters>
+                </plugin>
              </gazebo>
         </xacro:if>

Commit message: dd

File: robotiq_description/srdf/robotiq_2f_85_macro.srdf.xacro (robot description, xacro)
@@ -12,10 +12,4 @@
             <link name="${prefix}robotiq_85_right_finger_link"/>
             <link name="${prefix}robotiq_85_right_finger_tip_link"/>
-            <joint name="${prefix}robotiq_85_left_knuckle_joint" />
-            <passive_joint name="${prefix}robotiq_85_right_knuckle_joint" />
-            <passive_joint name="${prefix}robotiq_85_left_inner_knuckle_joint" />
-            <passive_joint name="${prefix}robotiq_85_right_inner_knuckle_joint" />
-            <passive_joint name="${prefix}robotiq_85_left_finger_tip_joint" />
-            <passive_joint name="${prefix}robotiq_85_right_finger_tip_joint" />
         </group>
         <!--GROUP STATES - Purpose - Define a named state for a particular group, in terms of joint values. This is useful to define states like 'folded arms'-->

File: robotiq_description/urdf/robotiq_2f_85_gripper.urdf.xacro (robot description, xacro)
@@ -2,5 +2,4 @@
 <robot xmlns:xacro="http://wiki.ros.org/xacro" name="robotiq_2f_85_gripper">
     <!-- parameters -->
-    <xacro:arg name="use_fake_hardware" default="false" />
     <xacro:arg name="sim_gazebo" default="false"/>
     <xacro:arg name="prefix" default="" />
@@ -11,5 +10,4 @@
         prefix="$(arg prefix)"
         parent="world"
-        use_fake_hardware="$(arg use_fake_hardware)"
         sim_gazebo="$(arg sim_gazebo)">
         <origin xyz="0 0 0.3" rpy="0 0 0" />
@@ -20,5 +18,5 @@
         <gazebo>
             <!-- gazebo ros2 control plugin -->
-            <plugin name="gazebo_ros_control" filename="libgazebo_ros2_control.so">
+            <plugin name="gazebo_ros2_control" filename="libgazebo_ros2_control.so">
                 <parameters>$(find robotiq_description)/config/robotiq_2f_85_controllers.yaml</parameters>
             </plugin>
